Commit message: Update rugved_description.urdf

File: rugved_description/urdf/rugved_description.urdf (robot description, URDF)
Before this commit: robot rugved_description, 5 links, 4 joints
Joints:
- joint horizontal_castor_joint: limit lower=-99999999999999999999999999999999999999999999999 upper=999999999999999999999999999999999999999999999999 effort=500 velocity=1 -> effort=500 velocity=1; type revolute -> continuous
- joint left_wheel_joint: limit lower=-99999999999999999999999999999999999999999999999 upper=999999999999999999999999999999999999999999999999 effort=1000 velocity=1 -> effort=1000 velocity=1; type revolute -> continuous
- joint right_wheel_joint: limit lower=-99999999999999999999999999999999999999999999999 upper=999999999999999999999999999999999999999999999999 effort=1000 velocity=1 -> effort=1000 velocity=1; type revolute -> continuous
- joint vertical_castor_joint: limit lower=-99999999999999999999999999999999999999999999999 upper=999999999999999999999999999999999999999999999999 effort=400 velocity=1 -> effort=400 velocity=1; type revolute -> continuous

Commit message: Update rugved_description.urdf

File: rugved_description/urdf/rugved_description.urdf (robot description, URDF)
Before this commit: robot rugved_description, 5 links, 4 joints
Links:
- added link hokuyo_link, mass 1e-5; collision box size=0.1 0.1 0.1; visual mesh filename=package://rugved_description/meshes/hokuyo.dae
Joints:
- added joint hokuyo_joint: type fixed, parent base_link, child hokuyo_link, origin xyz=0 0 0.7 rpy=0 0 0, axis 0 1 0
